File: hardware_dc/motoko_ice_dragon_x_dc.sch (EAGLE design)
At the start: 112 parts, among them IC2 A1202LH, IC3 A1202LH, IC4 A1202LH, IC5 A1202LH, J1 640-USB4105-GF-A-120, man. GCT, Q1 220mA/50V/3.5Ω, T1 FCX493TA, T2 BC847, U1 CH340E_MSOP10, U2 AP63203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

Commit message: documentation
Other:
- note added: "IMU"
- note added: "IR sensors"
- note added: "debug and interface"
- note added: "encoders"
- note added: "line sensors"
- note added: "microcontroller"
- note added: "motor drivers"
- note added: "power supply"
- note removed: "TS07-667-30-BK-160-SMT-TR"
- moved on the sheet: BATT, BOOT, C18, C20, C21, C22, C4, C5, C6, C7, D1, DEBUG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
