File: hardware/dc_motors copy/motoko_ice_dragon_x_dc.brd (EAGLE design)
At the start: 81.6 x 80 mm, 119 parts, among them IC2 A1202LH, IC3 A1202LH, IC4 A1202LH, IC5 A1202LH, J1 640-USB4105-GF-A-120, man. GCT, Q1 220mA/50V/3.5Ω, T1 FCX493TA, T2 BC847, U1 CP2102N, U2 AP63203, U3 STM32F722RET6, Y1 ABM8AIG-8.000MHZ-1Z-T

Commit message: encoder fix
Parts:
- removed C24: 100n, rcl:C0805
- removed C25: 10uF, rcl:C0805
- removed R36, R37, R38: 4k7, rcl:M0805
- removed SJ1, SJ2: (no value), jumper:SJ
- removed U$15, U$16, U$17, U$18, U$19, U$2, U$20, U$21: SFH3710, my_library:SFH710
- added LED11, LED12, LED13, LED14, LED15, LED16, LED17, LED18: (no value), led:CHIPLED_1206
- R9: value 4.7R -> 2.2R
- U1: value CP2102N -> CH340E_MSOP10; device SparkFun-IC-Comms:QFN24 -> SparkFun-IC-Comms:MSOP10
- moved TP2 13.0 mm to (28.3, 55.5)
- moved T1 8.90 mm to (30.5, 59.4), turned to 270 degrees
- moved R9 8.66 mm to (31.4, 55.5), turned to 180 degrees
- moved U1 5.88 mm to (29.0, 52.0)
- moved R10 3.88 mm to (37.5, 53.3)
- moved T2 3.02 mm to (35.4, 56.1), turned to 270 degrees
- moved LED3 2.24 mm to (57.0, 73.0)
- moved LED4 1.41 mm to (63.0, 63.0)
- moved R4 1.36 mm to (40.6, 63.3)
- moved LED10 1.00 mm to (59.0, 7.00)
- moved LED5 1.00 mm to (67.0, 53.0)
- moved LED6 1.00 mm to (68.0, 43.0)
- moved LED7 1.00 mm to (68.0, 37.0)
- moved LED8 1.00 mm to (67.0, 27.0)
- moved LED9 1.00 mm to (64.0, 17.0)
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Connections:
- removed net N$31: SJ1.1, U1.23
- removed net N$32: R38.2, U1.9
- removed net N$38: R36.1, R37.2, U1.8
- removed net VCCINT: C25.1, D1.A, J1.VBUS1, J1.VBUS2, R37.1
- net +3V3: now also U1.10; no longer C24.1, R38.1, U1.5, U1.6
- net ADC0: now also LED18.C; no longer U$21.P$1
- net ADC1: now also LED17.C; no longer U$20.P$1
- net ADC2: now also LED16.C; no longer U$19.P$1
- net ADC3: now also LED15.C; no longer U$18.P$1
- net ADC4: now also LED14.C; no longer U$17.P$1
- net ADC5: now also LED13.C; no longer U$16.P$1
- net ADC6: now also LED12.C; no longer U$15.P$1
- net ADC7: now also LED11.C; no longer U$2.P$1
- net BOOT: no longer SJ2.2
- net D+: now also U1.1; no longer U1.3
- net D-: now also U1.2; no longer U1.4
- net GND: now also LED11.A, LED12.A, LED13.A, LED14.A, LED15.A, LED16.A, LED17.A, LED18.A, U1.3; no longer C24.2, C25.2, R36.2, U$15.P$2, U$16.P$2, U$17.P$2, U$18.P$2, U$19.P$2, U$2.P$2, U$20.P$2, U$21.P$2, U1.2, U1.PAD
- net N$9: now also D1.A, J1.VBUS1, J1.VBUS2; no longer SJ2.1, U1.19
- net RESET: no longer SJ1.2
- net UART_RX: now also U1.8; no longer U1.21
- net UART_TX: now also U1.9; no longer U1.20
Routing:
- net VCCINT: track 53.0 -> 0.00 mm, vias 4 -> 0
- net BOOT: track 78.8 -> 43.2 mm, vias 2 -> 1
- net RESET: track 63.6 -> 28.1 mm, vias 3 -> 2
- net N$31: track 13.5 -> 0.00 mm, vias 1 -> 0
- net PWM_LEFT_B: track 55.9 -> 42.7 mm
- net UART_RX: track 41.0 -> 29.7 mm, vias 2 -> 1
- net PWM_LEFT_A: track 51.8 -> 40.7 mm
- net UART_TX: track 36.0 -> 26.2 mm
- net N$15: track 101.7 -> 111.4 mm
- net N$9: track 5.92 -> 14.6 mm, vias 1 -> 3
- net N$38: track 7.86 -> 0.00 mm, vias 1 -> 0
- net +3V3: track 409.3 -> 402.6 mm, vias 16 -> 15
- net N$14: track 10.7 -> 16.8 mm, vias 0 -> 2
- net GND: track 586.7 -> 591.5 mm, vias 105 -> 100
- net N$30: track 85.8 -> 81.7 mm
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