File: hardware/dc_motors copy/motoko_ice_dragon_x_dc.sch (EAGLE design)
At the start: 119 parts, among them IC2 A1202LH, IC3 A1202LH, IC4 A1202LH, IC5 A1202LH, J1 640-USB4105-GF-A-120, man. GCT, Q1 220mA/50V/3.5Ω, T1 FCX493TA, T2 BC847, U1 CP2102N, U2 AP63203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

Commit message: encoder fix
Parts:
- removed C24: 100n, rcl:C-EUC0805
- removed C25: 10uF, rcl:C-EUC0805
- removed R36, R37, R38: 4k7, rcl:R-EU_M0805
- removed SJ1, SJ2: (no value), jumper:SJ
- removed U$15, U$16, U$17, U$18, U$19, U$2, U$20, U$21: SFH3710, my_library:SFH3710
- added LED11, LED12, LED13, LED14, LED15, LED16, LED17, LED18: (no value), led:LEDCHIPLED_1206
- R9: value 4.7R -> 2.2R
- U1: value CP2102N -> CH340E_MSOP10; device SparkFun-IC-Comms:CP2102N -> SparkFun-IC-Comms:CH340E_MSOP10
Connections:
- removed net N$31: SJ1.1, U1.DTR
- removed net N$32: R38.2, U1.!RSTB
- removed net N$38: R36.1, R37.2, U1.VBUS
- removed net VCCINT: C25.1, D1.A, J1.VBUS, R37.1
- net +3V3: now also U1.V3, U1.VCC; no longer C24.1, R38.1, U1.VDD, U1.VIO, U1.VREGIN
- net ADC0: now also LED18.C; no longer U$21.C
- net ADC1: now also LED17.C; no longer U$20.C
- net ADC2: now also LED16.C; no longer U$19.C
- net ADC3: now also LED15.C; no longer U$18.C
- net ADC4: now also LED14.C; no longer U$17.C
- net ADC5: now also LED13.C; no longer U$16.C
- net ADC6: now also LED12.C; no longer U$15.C
- net ADC7: now also LED11.C; no longer U$2.C
- net BOOT: no longer SJ2.2
- net D+: now also U1.UD+; no longer U1.D+
- net D-: now also U1.UD-; no longer U1.D-
- net GND: now also LED11.A, LED12.A, LED13.A, LED14.A, LED15.A, LED16.A, LED17.A, LED18.A; no longer C24.2, C25.2, R36.2, U$15.E, U$16.E, U$17.E, U$18.E, U$19.E, U$2.E, U$20.E, U$21.E
- net N$9: now also D1.A, J1.VBUS; no longer SJ2.1, U1.RTS
- net RESET: no longer SJ1.2
- net UART_RX: now also U1.TXO; no longer U1.TXD
- net UART_TX: now also U1.RXI; no longer U1.RXD
