File: hardware/bldc_motors/motoko_ice_dragon_x_bldc.brd (EAGLE design)
At the start: 81.6 x 80 mm, 120 parts, among them J1 640-USB4105-GF-A-120, man. GCT, Q1 220mA/50V/3.5Ω, T1 FCX493TA, T2 BC847, U1 CH340E_MSOP10, U2 AP63203, U3 STM32F722RET6, Y1 ABM8AIG-8.000MHZ-1Z-T

Commit message: bldc test
Parts:
- removed U1: CH340E_MSOP10, SparkFun-IC-Comms:MSOP10
- added C29: 100n, rcl:C0805
- added C30: 10uF, rcl:C0805
- added R40, R41, R42: 4k7, rcl:M0805
- added SJ1, SJ2: (no value), jumper:SJ
- added U$5: (no value), my_library:DRAGON_LOGO_15MM
- added U4: CP2102N, SparkFun-IC-Comms:QFN24
- moved T1 9.76 mm to (37.2, 63.7), turned to 0 degrees
- moved TP2 6.01 mm to (40.5, 57.9), turned to 0 degrees
- moved T2 2.46 mm to (37.8, 56.4), turned to 180 degrees
- moved R4 1.36 mm to (41.8, 62.7)
- moved R10 1.22 mm to (38.7, 53.3), turned to 0 degrees
- moved R14 0.13 mm to (30.7, 28.5), turned to 0 degrees
- turned R9 to 0 degrees
Connections:
- net ENC_LEFT_A renamed ENC_LEFT_SCL
- net ENC_LEFT_B renamed ENC_LEFT_SDA
- net ENC_RIGHT_A renamed ENC_RIGHT_SCL
- net ENC_RIGHT_B renamed ENC_RIGHT_SDA
- removed net N$9: D1.A, J1.VBUS1, J1.VBUS2
- new net N$33: SJ1.1, U4.23
- new net N$34: SJ2.1, U4.19
- new net N$37: R40.2, U4.9
- new net N$38: R41.1, R42.2, U4.8
- new net VBUS: C30.1, D1.A, J1.VBUS1, J1.VBUS2, R42.1
- net +3V3: now also C29.1, R14.2, R40.1, U4.5, U4.6, U4.7; no longer BOOT.2, U1.10, U1.7
- net BOOT: now also BOOT.2, R14.1, SJ2.2; no longer BOOT.1, R14.2
- net D+: now also U4.3; no longer U1.1
- net D-: now also U4.4; no longer U1.2
- net GND: now also BOOT.1, C29.2, C30.2, R41.2, U4.2, U4.PAD; no longer R14.1, U1.3
- net RESET: now also SJ1.2
- net UART_RX: now also U4.21; no longer U1.8
- net UART_TX: now also U4.20; no longer U1.9
Routing:
- net VBUS: track 0.00 -> 47.5 mm, vias 0 -> 3
- net +3V3: track 417.1 -> 385.6 mm, vias 12 -> 13
- net BOOT: track 49.9 -> 75.1 mm, vias 2 -> 3
- net RESET: track 28.1 -> 53.0 mm, vias 2 -> 3
- net N$9: track 14.6 -> 0.00 mm, vias 3 -> 0
- net N$15: track 114.4 -> 102.0 mm
- net GND: track 674.1 -> 685.5 mm, vias 92 -> 87
- net UART_TX: track 26.2 -> 37.4 mm, vias 2 -> 3
- net N$33: track 0.00 -> 11.1 mm, vias 0 -> 1
- net UART_RX: track 29.7 -> 39.5 mm, vias 1 -> 3
- net D+: track 37.1 -> 42.3 mm
- net N$37: track 0.00 -> 4.90 mm
- net N$38: track 0.00 -> 4.42 mm, vias 0 -> 1
- net N$14: track 7.14 -> 10.3 mm
- net N$34: track 0.00 -> 3.15 mm, vias 0 -> 1
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Other:
- board size 81.6 x 80 mm -> 81 x 80 mm
