File: hardware/bldc_motors/motoko_ice_dragon_x_bldc.sch (EAGLE design)
At the start: 120 parts, among them J1 640-USB4105-GF-A-120, man. GCT, Q1 220mA/50V/3.5Ω, T1 FCX493TA, T2 BC847, U1 CH340E_MSOP10, U2 AP63203, U3 STM32F722RET6, Y1 ABM8AIG-8.000MHZ-1Z-T

Commit message: bldc test
Parts:
- removed U1: CH340E_MSOP10, SparkFun-IC-Comms:CH340E_MSOP10
- added C29: 100n, rcl:C-EUC0805
- added C30: 10uF, rcl:C-EUC0805
- added R40, R41, R42: 4k7, rcl:R-EU_M0805
- added SJ1, SJ2: (no value), jumper:SJ
- added U4: CP2102N, SparkFun-IC-Comms:CP2102N
Connections:
- net ENC_LEFT_A renamed ENC_LEFT_SCL
- net ENC_LEFT_B renamed ENC_LEFT_SDA
- net ENC_RIGHT_A renamed ENC_RIGHT_SCL
- net ENC_RIGHT_B renamed ENC_RIGHT_SDA
- removed net N$9: D1.A, J1.VBUS
- new net N$33: SJ1.1, U4.DTR
- new net N$34: SJ2.1, U4.RTS
- new net N$37: R40.2, U4.!RSTB
- new net N$38: R41.1, R42.2, U4.VBUS
- new net VBUS: C30.1, D1.A, J1.VBUS, R42.1
- net +3V3: now also C29.1, R14.2, R40.1, U4.VDD, U4.VIO, U4.VREGIN; no longer BOOT.2, U1.V3, U1.VCC
- net BOOT: now also BOOT.2, R14.1, SJ2.2; no longer BOOT.1, R14.2
- net D+: now also U4.D+; no longer U1.UD+
- net D-: now also U4.D-; no longer U1.UD-
- net GND: now also BOOT.1, C29.2, C30.2, R41.2, U4.GND; no longer R14.1, U1.GND
- net RESET: now also SJ1.2
- net UART_RX: now also U4.TXD; no longer U1.TXO
- net UART_TX: now also U4.RXD; no longer U1.RXI
Other:
- moved on the sheet: BOOT, C20, C21, C22, R14, U3B, Y1
