File: hardware/dc_motors/motoko_ice_dragon_x_dc.sch (EAGLE design)
At the start: 119 parts, among them IC2 A1202LH, IC3 A1202LH, IC4 A1202LH, IC5 A1202LH, J1 640-USB4105-GF-A-120, man. GCT, Q1 220mA/50V/3.5Ω, T1 FCX493TA, T2 BC847, U1 CP2102N, U2 AP63203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

Commit message: bldc test
Other:
- moved on the sheet: C20, C21, C22, C24, C25, R36, R37, R38, SJ1, SJ2, U1, U3B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
